File: PCBs/FineMotion-5.kicad_pcb (KiCad board)
At the start: 2 copper layers, 49.3 x 19.7 mm, 43 parts, among them J1 Conn_01x02_Female, J2 Conn_01x04_Female, P1 USB_C_Plug_USB2.0, SW1 Option/FLASH Switch, SW3 SW_SPDT MAIN POWER, U1 ME6211C, U2 TP4056, U6 ESP-12F, U7 CH340C, U9 MPU-9250

Commit message: bmi160
Parts:
- removed C7: 0.1uF, Capacitor_SMD:C_0402_1005Metric
- removed U9: MPU-9250, Sensor_Motion:InvenSense_QFN-24_3x3mm_P0.4mm
- added U3: BMI160, Package_LGA:Bosch_LGA-14_3x2.5mm_P0.5mm, F.Cu at (118.9, 65.8)
- renumbered C2 to C3, R12 to R3, R11 to R7
Routing:
- net GND: track 163.0 -> 151.0 mm, vias 47 -> 45
- net Net-(C7-Pad1): track 1.22 -> 0.00 mm
Other:
- board text added: "BMI160"
- board text removed: "MPU6500"
